File: UFO/UFO.kicad_pcb (KiCad board)
At the start: 2 copper layers, 390.9 x 114.4 mm, 345 parts, among them U1 Raspberry_Pi_Pico

Commit message: ufo v1.1 with case (the version that I had made)
Parts:
- added REF**: MountingHole_4mm, MountingHole:MountingHole_4mm, F.Cu at (159.6, 95.5)
- added REF**: MountingHole_4mm, MountingHole:MountingHole_4mm, F.Cu at (292.9, 95.5)
- added REF**: MountingHole_4mm, MountingHole:MountingHole_4mm, F.Cu at (159.6, 57.4)
- added REF**: MountingHole_4mm, MountingHole:MountingHole_4mm, F.Cu at (292.9, 57.4)
- moved D34 4.29 mm to (158.3, 88.5)
- moved D74 2.94 mm to (291.7, 51.8)
- moved D32 2.35 mm to (158.5, 52.4)
- moved D76 1.79 mm to (291.7, 91.0)
- moved D114 0.87 mm to (405.5, 130.2)
- moved D113 0.31 mm to (405.6, 111.9)
- moved D112 0.21 mm to (405.8, 92.8)
Routing:
- net GND: track 3032.3 -> 3026.1 mm
- net Row 3: track 399.5 -> 404.5 mm
- net Row 1: track 370.8 -> 375.2 mm
- net Net-(D34-A): track 11.3 -> 7.07 mm
- net Col 6: track 289.9 -> 293.4 mm
- net Net-(D153-DOUT): track 386.2 -> 389.4 mm
- net Col 7: track 307.2 -> 310.3 mm
- net Col 8: track 324.9 -> 328.0 mm
- net Net-(D74-A): track 11.3 -> 8.42 mm
- net Net-(D32-A): track 11.3 -> 9.08 mm
- net Net-(D76-A): track 11.3 -> 9.57 mm
- net Net-(D146-DOUT): track 15.3 -> 14.3 mm
- net Net-(D182-DOUT): track 15.2 -> 14.3 mm
- net Net-(D139-DOUT): track 15.2 -> 14.3 mm
- net Row 5: track 680.2 -> 681.0 mm
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Other:
- board size 390.9 x 114.4 mm -> 388.1 x 114.4 mm
