File: UFO/rgbled.kicad_sch (KiCad schematic)
At the start: 114 parts

Commit message: ufo v1.1 with case (the version that I had made)
Other:
- title: (none) -> RGB Matrix
Changed lines of the file:
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@@
 	(generator_version "8.0")
 	(paper "A3")
+	(title_block
+		(title "RGB Matrix")
+		(date "2025-07-25")
+		(rev "1")
+	)
 	(junction
 		(at 265.43 115.57)
